File: CustomPCB/PowerPCB/PowerPCB.kicad_pcb (KiCad board)
At the start: 2 copper layers, 100 x 40 mm, 16 parts, among them J1 XT30, J2 XT60, J3 Barrel_Jack_15V, J4 Barrel_Jack_5V, U1 LM1084-ADJ, U2 LM1084-5.0

Commit message: costum pcb update
#19
Parts:
- added H1: MountingHole, MountingHole:MountingHole_2.5mm, F.Cu at (118.0, 63.0)
- added H2: MountingHole, MountingHole:MountingHole_2.5mm, F.Cu at (171.0, 63.0)
- added H3: MountingHole, MountingHole:MountingHole_2.5mm, F.Cu at (118.0, 93.0)
- added H4: MountingHole, MountingHole:MountingHole_2.5mm, F.Cu at (171.0, 93.0)
Routing:
- net (no net): vias 4 -> 0

Commit message: update PowerPCB
#19
Parts:
- moved H1 1.90 mm to (116.2, 62.2)
- moved H3 1.90 mm to (116.2, 93.8)
- moved H2 1.46 mm to (169.8, 62.2)
- moved H4 1.46 mm to (169.8, 93.8)
Changed lines of the file:
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@@
   )
   (footprint "MountingHole:MountingHole_2.5mm" (layer "F.Cu")
-    (at 118 63)
+    (at 116.25 62.25)
     (descr "Mounting Hole 2.5mm, no annular")
     (tags "mounting hole 2.5mm no annular")
@@
   )
   (footprint "MountingHole:MountingHole_2.5mm" (layer "F.Cu")
-    (at 171 63)
+    (at 169.75 62.25)
     (descr "Mounting Hole 2.5mm, no annular")
     (tags "mounting hole 2.5mm no annular")
@@
   )
   (footprint "MountingHole:MountingHole_2.5mm" (layer "F.Cu")
-    (at 118 93)
+    (at 116.25 93.75)
     (descr "Mounting Hole 2.5mm, no annular")
     (tags "mounting hole 2.5mm no annular")
@@
   )
   (footprint "MountingHole:MountingHole_2.5mm" (layer "F.Cu")
-    (at 171 93)
+    (at 169.75 93.75)
     (descr "Mounting Hole 2.5mm, no annular")
     (tags "mounting hole 2.5mm no annular")

Commit message: updates
#23 #20
Parts:
- J3, J4: footprint Connector_BarrelJack:BarrelJack_CUI_PJ-102AH_Horizontal -> Connector_BarrelJack:BarrelJack_CUI_PJ-102AH_Horizontal_flat_pins
