File: CustomPCB/PowerPCB/PowerPCB.kicad_sch (KiCad schematic)
At the start: 16 parts, among them J1 XT30, J2 XT60, J3 Barrel_Jack_15V, J4 Barrel_Jack_5V, U1 LM1084-ADJ, U2 LM1084-5.0

Commit message: costum pcb update
#19
Parts:
- added H1, H2, H3, H4: MountingHole, MountingHole:MountingHole_2.5mm, symbol Mechanical:MountingHole
Changed lines of the file:
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@@
     (pin "3")
+  )
+  (symbol (lib_id "Mechanical:MountingHole") (at 180.34 50.8 0) (unit 1)
+    (in_bom yes) (on_board yes)
+    (property "Reference" "H1" (id 0) (at 182.88 49.5299 0)
+      (effects (font (size 1.27 1.27)) (justify left))
+    )
+    (property "Value" "MountingHole" (id 1) (at 182.88 45.72 0)
+      (effects (font (size 1.27 1.27)) (justify left))
+    )
+    (property "Footprint" "MountingHole:MountingHole_2.5mm" (id 2) (at 180.34 50.8 0)
+      (effects (font (size 1.27 1.27)) hide)
+    )
+    (property "Datasheet" "~" (id 3) (at 180.34 50.8 0)
+      (effects (font (size 1.27 1.27)) hide)
+    )
   )
   (symbol (lib_id "power:GND") (at 64.77 69.85 0) (mirror y) (unit 1)
@@
     (pin "2")
     (pin "3")
+  )
+  (symbol (lib_id "Mechanical:MountingHole") (at 190.5 55.88 0) (unit 1)
+    (in_bom yes) (on_board yes) (fields_autoplaced)
+    (property "Reference" "H4" (id 0) (at 193.04 54.6099 0)
+      (effects (font (size 1.27 1.27)) (justify left))
+    )
+    (property "Value" "MountingHole" (id 1) (at 193.04 57.1499 0)
+      (effects (font (size 1.27 1.27)) (justify left) hide)
+    )
+    (property "Footprint" "MountingHole:MountingHole_2.5mm" (id 2) (at 190.5 55.88 0)
+      (effects (font (size 1.27 1.27)) hide)
+    )
+    (property "Datasheet" "~" (id 3) (at 190.5 55.88 0)
+      (effects (font (size 1.27 1.27)) hide)
+    )
   )
   (symbol (lib_id "Device:C_Polarized") (at 88.9 96.52 0) (unit 1)
@@
     )
     (pin "1")
+  )
+  (symbol (lib_id "Mechanical:MountingHole") (at 180.34 55.88 0) (unit 1)
+    (in_bom yes) (on_board yes)
+    (property "Reference" "H2" (id 0) (at 182.88 54.6099 0)
+      (effects (font (size 1.27 1.27)) (justify left))
+    )
+    (property "Value" "MountingHole" (id 1) (at 182.88 55.8799 0)
+      (effects (font (size 1.27 1.27)) (justify left) hide)
+    )
+    (property "Footprint" "MountingHole:MountingHole_2.5mm" (id 2) (at 180.34 55.88 0)
+      (effects (font (size 1.27 1.27)) hide)
+    )
+    (property "Datasheet" "~" (id 3) (at 180.34 55.88 0)
+      (effects (font (size 1.27 1.27)) hide)
+    )
+  )
+  (symbol (lib_id "Mechanical:MountingHole") (at 190.5 50.8 0) (unit 1)
+    (in_bom yes) (on_board yes)
+    (property "Reference" "H3" (id 0) (at 193.04 49.5299 0)
+      (effects (font (size 1.27 1.27)) (justify left))
+    )
+    (property "Value" "MountingHole" (id 1) (at 193.04 50.7999 0)
+      (effects (font (size 1.27 1.27)) (justify left) hide)
+    )
+    (property "Footprint" "MountingHole:MountingHole_2.5mm" (id 2) (at 190.5 50.8 0)
+      (effects (font (size 1.27 1.27)) hide)
+    )
+    (property "Datasheet" "~" (id 3) (at 190.5 50.8 0)
+      (effects (font (size 1.27 1.27)) hide)
+    )
   )
   (symbol (lib_id "Connector:Barrel_Jack_MountingPin") (at 176.53 78.74 0) (mirror y) (unit 1)
@@
       (effects (font (size 1.27 1.27)) hide)
     )
-    (pin "2")
-    (pin "1")
+    (pin "1")
+    (pin "2")
   )
   (symbol (lib_id "power:GND") (at 105.41 69.85 0) (unit 1)
@@
       (reference "D1") (unit 1) (value "1N4007") (footprint "Diode_THT:D_DO-41_SOD81_P10.16mm_Horizontal")
     )
+    (path "/1533b475-c834-40d3-ae2c-55eb46ae810f"
+      (reference "H1") (unit 1) (value "MountingHole") (footprint "MountingHole:MountingHole_2.5mm")
+    )
+    (path "/8fac398c-22c9-4741-a001-aab7ea92da04"
+      (reference "H2") (unit 1) (value "MountingHole") (footprint "MountingHole:MountingHole_2.5mm")
+    )
+    (path "/9d5e7df5-7472-4dc8-a9fc-73987a422b16"
+      (reference "H3") (unit 1) (value "MountingHole") (footprint "MountingHole:MountingHole_2.5mm")
+    )
+    (path "/2b105527-e599-4635-9472-cb4bb39953cd"
+      (reference "H4") (unit 1) (value "MountingHole") (footprint "MountingHole:MountingHole_2.5mm")
+    )
     (path "/2979e3a0-3605-49e3-aa66-4b2a3861df27"

Commit message: updates
#23 #20
Parts:
- J3, J4: footprint Connector_BarrelJack:BarrelJack_CUI_PJ-102AH_Horizontal -> Connector_BarrelJack:BarrelJack_CUI_PJ-102AH_Horizontal_flat_pins
Changed lines of the file:
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@@
     (property "Reference" "J3" (id 0) (at 105.41 50.8 0))
     (property "Value" "Barrel_Jack_15V" (id 1) (at 105.41 53.34 0))
-    (property "Footprint" "Connector_BarrelJack:BarrelJack_CUI_PJ-102AH_Horizontal" (id 2) (at 106.68 60.706 0)
+    (property "Footprint" "Connector_BarrelJack:BarrelJack_CUI_PJ-102AH_Horizontal_flat_pins" (id 2) (at 106.68 60.706 0)
       (effects (font (size 1.27 1.27)) hide)
     )
@@
       (effects (font (size 1.27 1.27)) (justify right))
     )
-    (property "Footprint" "Connector_BarrelJack:BarrelJack_CUI_PJ-102AH_Horizontal" (id 2) (at 175.26 79.756 0)
+    (property "Footprint" "Connector_BarrelJack:BarrelJack_CUI_PJ-102AH_Horizontal_flat_pins" (id 2) (at 175.26 79.756 0)
       (effects (font (size 1.27 1.27)) hide)
     )
@@
     )
     (path "/5e32da30-1a3e-4135-adaf-bbf389b0c3fc"
-      (reference "J3") (unit 1) (value "Barrel_Jack_15V") (footprint "Connector_BarrelJack:BarrelJack_CUI_PJ-102AH_Horizontal")
+      (reference "J3") (unit 1) (value "Barrel_Jack_15V") (footprint "Connector_BarrelJack:BarrelJack_CUI_PJ-102AH_Horizontal_flat_pins")
     )
     (path "/a1230e51-a25e-405f-a529-6d77ce24c790"
-      (reference "J4") (unit 1) (value "Barrel_Jack_5V") (footprint "Connector_BarrelJack:BarrelJack_CUI_PJ-102AH_Horizontal")
+      (reference "J4") (unit 1) (value "Barrel_Jack_5V") (footprint "Connector_BarrelJack:BarrelJack_CUI_PJ-102AH_Horizontal_flat_pins")
     )
     (path "/6b7ed168-4871-4946-bdda-64b58286ec65"
